Commit message: Added a prismatic joint for grasp center planning Fixed setup assistant config

File: sr_multi_description/urdf/shadow_ur10.urdf.xacro (robot description, xacro)
@@ -18,8 +18,10 @@
       <origin xyz="0.012 0.0 0.0" rpy="${pi/2.0} ${pi} ${pi/2.0}" />
     </joint>
-  <joint name="arm_to_hand" type="float">
+  <joint name="hand_to_grasp" type="prismatic">
       <parent link="palm" />
       <child link="grasp_center" />
       <origin xyz="0.0 -0.08 0.09" rpy="0.0 0.0 0.0" />
+      <axis xyz="0 -1 0" />
+      <limit lower="-0.08" upper="0.08" effort="30" velocity="2.0" />
     </joint>
   <link name="grasp_center"/>

File: sr_multi_description/urdf/shadow_ur10_joint_limited.urdf.xacro (robot description, xacro)
@@ -18,3 +18,11 @@
       <origin xyz="0.012 0.0 0.0" rpy="${pi/2.0} ${pi} ${pi/2.0}" />
     </joint>
+  <joint name="hand_to_grasp" type="prismatic">
+      <parent link="palm" />
+      <child link="grasp_center" />
+      <origin xyz="0.0 -0.08 0.09" rpy="0.0 0.0 0.0" />
+      <axis xyz="0 -1 0" />
+      <limit lower="-0.08" upper="0.08" effort="30" velocity="2.0" />
+    </joint>
+  <link name="grasp_center"/>
  </robot>

Commit message: Created a binamual system in namespaces, and disable the virtual grasp center Adapted moveit to use trajectory controllers in namespaces

File: sr_multi_description/urdf/shadow_ur10.urdf.xacro (robot description, xacro)
@@ -1,4 +1,3 @@
  <robot xmlns:xacro="http://ros.org/wiki/xacro" name="ur10shadow">
-  <!--<xacro:include filename="$(find ur_description)/urdf/gazebo.urdf.xacro" />-->
   <xacro:include filename="$(find ur_description)/urdf/ur10.urdf.xacro" />
   <link name="world" />
@@ -8,14 +7,21 @@
     <origin xyz="0.0 0.0 0.0" rpy="0.0 0.0 0.0" />
   </joint>
+  <!-- instantiate the arm -->
   <xacro:ur10_robot prefix="" joint_limited="false"/>
+  <!-- add the plugin which will be in a namespace (arm) -->
+  <xacro:include filename="$(find sr_multi_description)/urdf/ur_gazebo.urdf.xacro" />
   <xacro:include filename="$(find sr_description)/materials.urdf.xacro" />
   <xacro:include filename="$(find sr_description)/hand/xacro/full_hand.urdf.xacro" />
-  <xacro:include filename="$(find sr_description)/other/xacro/gazebo/gazebo.urdf.xacro" />
+  <!-- instantiate the hand -->
   <xacro:shadowhand muscletrans="false" muscle="false" bio="false" bt_sp="false" ubi="false" eli="false" reflect="1.0" prefix="" />
-    <joint name="arm_to_hand" type="fixed">
-      <parent link="ee_link" />
-      <child link = "forearm" />
-      <origin xyz="0.012 0.0 0.0" rpy="${pi/2.0} ${pi} ${pi/2.0}" />
-    </joint>
+  <!-- add the plugin which will be in a namespace (hand) -->
+  <xacro:include filename="$(find sr_multi_description)/urdf/sr_gazebo.urdf.xacro" />
+  <!-- attach the hand to the arm -->
+  <joint name="arm_to_hand" type="fixed">
+    <parent link="ee_link" />
+    <child link = "forearm" />
+    <origin xyz="0.012 0.0 0.0" rpy="${pi/2.0} ${pi} ${pi/2.0}" />
+  </joint>
+ <!-- virtual link for grasping
   <joint name="hand_to_grasp" type="prismatic">
       <parent link="palm" />
@@ -25,4 +31,4 @@
       <limit lower="-0.08" upper="0.08" effort="30" velocity="2.0" />
     </joint>
-  <link name="grasp_center"/>
+  <link name="grasp_center"/>-->
  </robot>

File: sr_multi_description/urdf/shadow_ur10_joint_limited.urdf.xacro (robot description, xacro)
@@ -1,4 +1,3 @@
  <robot xmlns:xacro="http://ros.org/wiki/xacro" name="ur10shadow">
-  <!--<xacro:include filename="$(find ur_description)/urdf/gazebo.urdf.xacro" />-->
   <xacro:include filename="$(find ur_description)/urdf/ur10.urdf.xacro" />
   <link name="world" />
@@ -8,14 +7,21 @@
     <origin xyz="0.0 0.0 0.0" rpy="0.0 0.0 0.0" />
   </joint>
+  <!-- instantiate the arm -->
   <xacro:ur10_robot prefix="" joint_limited="true"/>
+  <!-- add the plugin which will be in a namespace (arm) -->
+  <xacro:include filename="$(find sr_multi_description)/urdf/ur_gazebo.urdf.xacro" />
   <xacro:include filename="$(find sr_description)/materials.urdf.xacro" />
   <xacro:include filename="$(find sr_description)/hand/xacro/full_hand.urdf.xacro" />
-  <xacro:include filename="$(find sr_description)/other/xacro/gazebo/gazebo.urdf.xacro" />
+  <!-- instantiate the hand -->
   <xacro:shadowhand muscletrans="false" muscle="false" bio="false" bt_sp="false" ubi="false" eli="false" reflect="1.0" prefix="" />
-    <joint name="arm_to_hand" type="fixed">
-      <parent link="ee_link" />
-      <child link = "forearm" />
-      <origin xyz="0.012 0.0 0.0" rpy="${pi/2.0} ${pi} ${pi/2.0}" />
-    </joint>
+  <!-- add the plugin which will be in a namespace (hand) -->
+  <xacro:include filename="$(find sr_multi_description)/urdf/sr_gazebo.urdf.xacro" />
+  <!-- attach the hand to the arm -->
+  <joint name="arm_to_hand" type="fixed">
+    <parent link="ee_link" />
+    <child link = "forearm" />
+    <origin xyz="0.012 0.0 0.0" rpy="${pi/2.0} ${pi} ${pi/2.0}" />
+  </joint>
+ <!-- virtual link for grasping
   <joint name="hand_to_grasp" type="prismatic">
       <parent link="palm" />
@@ -25,4 +31,4 @@
       <limit lower="-0.08" upper="0.08" effort="30" velocity="2.0" />
     </joint>
-  <link name="grasp_center"/>
+  <link name="grasp_center"/>-->
  </robot>
